File: sch_pcb/LED Pong.kicad_pcb (KiCad board)
At the start: 2 copper layers, 69.6 x 54.4 mm, 14 parts, among them SW1 SW_Push, SW2 SW_Push

Commit message: update brd
Parts:
- A1: moved to B.Cu
- moved A1 48.0 mm to (132.0, 119.1)
- moved BZ1 10.7 mm to (110.0, 79.8)
- moved SW2 2.34 mm to (110.8, 107.0)
- moved D8 1.79 mm to (115.8, 93.5)
- moved D1 1.78 mm to (168.9, 93.5)
- moved D2 1.78 mm to (161.3, 93.5)
- moved D3 1.78 mm to (153.7, 93.5)
- moved D4 1.78 mm to (146.1, 93.5)
- moved D5 1.78 mm to (138.5, 93.5)
- moved D6 1.78 mm to (130.8, 93.5)
- moved D7 1.78 mm to (123.2, 93.5)
- moved D9 1.78 mm to (108.0, 93.5)
Routing:
- net GND: track 187.9 -> 0.00 mm
- net Net-(A1-D2): track 122.7 -> 0.00 mm
- net Net-(D1-K): track 73.9 -> 0.00 mm
- net Net-(A1-D4): track 59.1 -> 0.00 mm
- net /D13: track 43.9 -> 0.00 mm
- net /D12: track 38.8 -> 0.00 mm
- net /D5: track 37.8 -> 0.00 mm
- net /D11: track 36.4 -> 0.00 mm
- net /D6: track 31.5 -> 0.00 mm
- net /D10: track 31.0 -> 0.00 mm
- net /D9: track 27.1 -> 0.00 mm
- net /D7: track 26.7 -> 0.00 mm
- net /D8: track 25.3 -> 0.00 mm
- net Net-(A1-D3): track 15.6 -> 0.84 mm
Other:
- board size 69.6 x 54.4 mm -> 69.1 x 53.8 mm

Commit message: update brd
Parts:
- moved R1 6.28 mm to (131.1, 80.3), turned to 180 degrees
- moved BZ1 4.76 mm to (110.6, 75.0), turned to -45 degrees
- moved D8 2.84 mm to (115.3, 96.3), turned to 90 degrees
- moved D2 2.81 mm to (161.0, 96.3), turned to 90 degrees
- moved D3 2.81 mm to (153.4, 96.3), turned to 90 degrees
- moved D4 2.81 mm to (145.8, 96.3), turned to 90 degrees
- moved D5 2.81 mm to (138.2, 96.3), turned to 90 degrees
- moved D7 2.81 mm to (122.9, 96.3), turned to 90 degrees
- moved D9 2.81 mm to (107.7, 96.3), turned to 90 degrees
- moved D1 2.81 mm to (168.7, 96.3), turned to 90 degrees
- moved D6 2.81 mm to (130.6, 96.3), turned to 90 degrees
Routing:
- net Net-(A1-D4): track 0.00 -> 97.1 mm
- net Net-(D1-K): track 0.00 -> 81.0 mm
- net Net-(A1-D3): track 0.84 -> 55.7 mm
- net Net-(A1-D2): track 0.00 -> 54.7 mm
- net /D13: track 0.00 -> 35.7 mm
- net /D12: track 0.00 -> 31.0 mm
- net /D11: track 0.00 -> 28.2 mm
- net /D5: track 0.00 -> 27.6 mm
- net /D10: track 0.00 -> 25.5 mm
- net /D6: track 0.00 -> 25.1 mm
- net /D9: track 0.00 -> 24.1 mm
- net /D7: track 0.00 -> 23.8 mm
- net /D8: track 0.00 -> 22.9 mm
- added copper zone on B.Cu, net GND

Commit message: update pcb
Routing:
- net Net-(D1-K): track 81.0 -> 81.7 mm

Commit message: update pcb
Routing:
- net /D13: track 35.7 -> 37.1 mm
Changed lines of the file:
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@@
   (arc (start 117.788629 69.088) (mid 116.64058 69.316359) (end 115.667308 69.96668) (width 1) (layer "B.Cu") (net 16))
   (arc (start 159.412359 69.088) (mid 160.560409 69.316361) (end 161.533679 69.966679) (width 1) (layer "B.Cu") (net 16))
-  (segment (start 159.31 111.4552) (end 159.7152 111.4552) (width 1) (layer "B.Cu") (net 17))
-  (segment (start 159.31 111.4552) (end 165.81 111.4552) (width 1) (layer "B.Cu") (net 17))
-  (segment (start 165.81 111.4552) (end 166.728591 111.4552) (width 1) (layer "B.Cu") (net 17))
-  (segment (start 171.704 105.330319) (end 171.704 87.884) (width 1) (layer "B.Cu") (net 17))
-  (segment (start 159.7152 111.4552) (end 160.02 111.76) (width 1) (layer "B.Cu") (net 17))
-  (segment (start 162.138064 76.286064) (end 170.267158 84.415158) (width 1) (layer "B.Cu") (net 17))
-  (arc (start 170.267158 84.415158) (mid 171.330576 86.006675) (end 171.704 87.884) (width 1) (layer "B.Cu") (net 17))
-  (arc (start 169.672 110.236) (mid 171.1759 107.985254) (end 171.704 105.330319) (width 1) (layer "B.Cu") (net 17))
-  (arc (start 159.893 70.866) (mid 160.476473 73.799317) (end 162.138064 76.286064) (width 1) (layer "B.Cu") (net 17))
-  (arc (start 166.728591 111.4552) (mid 168.321552 111.138341) (end 169.672 110.236) (width 1) (layer "B.Cu") (net 17))
+  (segment (start 159.31 111.4552) (end 159.7152 111.4552) (width 0.75) (layer "B.Cu") (net 17))
+  (segment (start 159.31 111.4552) (end 165.81 111.4552) (width 0.75) (layer "B.Cu") (net 17))
+  (segment (start 165.81 111.4552) (end 166.728591 111.4552) (width 0.75) (layer "B.Cu") (net 17))
+  (segment (start 171.704 105.330319) (end 171.704 87.884) (width 0.75) (layer "B.Cu") (net 17))
+  (segment (start 159.7152 111.4552) (end 160.02 111.76) (width 0.75) (layer "B.Cu") (net 17))
+  (segment (start 162.138064 76.286064) (end 170.267158 84.415158) (width 0.75) (layer "B.Cu") (net 17))
+  (arc (start 170.267158 84.415158) (mid 171.330576 86.006675) (end 171.704 87.884) (width 0.75) (layer "B.Cu") (net 17))
+  (arc (start 169.672 110.236) (mid 171.1759 107.985254) (end 171.704 105.330319) (width 0.75) (layer "B.Cu") (net 17))
+  (arc (start 159.893 70.866) (mid 160.476473 73.799317) (end 162.138064 76.286064) (width 0.75) (layer "B.Cu") (net 17))
+  (arc (start 166.728591 111.4552) (mid 168.321552 111.138341) (end 169.672 110.236) (width 0.75) (layer "B.Cu") (net 17))
   (segment (start 169.672 100.584) (end 169.242754 101.013246) (width 0.75) (layer "B.Cu") (net 18))
   (segment (start 128.249584 106.954416) (end 131.064 104.14) (width 0.75) (layer "B.Cu") (net 18))
   (segment (start 170.688 92.789681) (end 170.688 98.552) (width 0.75) (layer "B.Cu") (net 18))
   (segment (start 169.96958 100.286421) (end 169.672 100.584) (width 0.75) (layer "B.Cu") (net 18))
-  (segment (start 110.848 111.47) (end 117.348 111.47) (width 1.25) (layer "B.Cu") (net 18))
+  (segment (start 110.848 111.47) (end 117.348 111.47) (width 0.75) (layer "B.Cu") (net 18))
   (segment (start 137.196102 101.6) (end 167.413359 101.6) (width 0.75) (layer "B.Cu") (net 18))
   (segment (start 168.656 87.884) (end 161.394099 80.622099) (width 0.75) (layer "B.Cu") (net 18))
@@
   (segment (start 135.513 72.291359) (end 135.513 70.866) (width 1) (layer "B.Cu") (net 26))
   (arc (start 135.513 72.291359) (mid 135.284639 73.439409) (end 134.634321 74.412679) (width 1) (layer "B.Cu") (net 26))
-  (segment (start 109.43042 91.948) (end 112.461903 91.948) (width 1) (layer "B.Cu") (net 27))
-  (segment (start 107.696 93.731) (end 107.696 93.68242) (width 1) (layer "B.Cu") (net 27))
-  (segment (start 114.583224 91.06932) (end 131.69063 73.961914) (width 1) (layer "B.Cu") (net 27))
-  (arc (start 131.69063 73.961914) (mid 132.639724 72.541498) (end 132.973 70.866) (width 1) (layer "B.Cu") (net 27))
-  (arc (start 112.461903 91.948) (mid 113.609954 91.719639) (end 114.583224 91.06932) (width 1) (layer "B.Cu") (net 27))
-  (arc (start 108.204 92.456) (mid 108.766686 92.080025) (end 109.43042 91.948) (width 1) (layer "B.Cu") (net 27))
-  (arc (start 107.696 93.68242) (mid 107.828025 93.018687) (end 108.204 92.456) (width 1) (layer "B.Cu") (net 27))
+  (segment (start 107.696 93.731) (end 107.696 92.362214) (width 1) (layer "B.Cu") (net 27))
+  (segment (start 107.988893 91.655107) (end 108.126214 91.517786) (width 1) (layer "B.Cu") (net 27))
+  (segment (start 116.70268 90.05332) (end 132.094321 74.661679) (width 1) (layer "B.Cu") (net 27))
+  (segment (start 109.540427 90.932) (end 114.581359 90.932) (width 1) (layer "B.Cu") (net 27))
+  (segment (start 132.973 72.540359) (end 132.973 70.866) (width 1) (layer "B.Cu") (net 27))
+  (arc (start 108.126214 91.517786) (mid 108.77506 91.084241) (end 109.540427 90.932) (width 1) (layer "B.Cu") (net 27))
+  (arc (start 116.70268 90.05332) (mid 115.72941 90.703639) (end 114.581359 90.932) (width 1) (layer "B.Cu") (net 27))
+  (arc (start 107.988893 91.655107) (mid 107.77212 91.97953) (end 107.696 92.362214) (width 1) (layer "B.Cu") (net 27))
+  (arc (start 132.094321 74.661679) (mid 132.744639 73.688409) (end 132.973 72.540359) (width 1) (layer "B.Cu") (net 27))
   (segment (start 118.872 96.271) (end 107.696 96.271) (width 1.25) (layer "B.Cu") (net 31))
   (segment (start 168.656 96.271) (end 119.888 96.271) (width 1.25) (layer "B.Cu") (net 31))

Commit message: update pcb
Parts:
- A1: footprint Module:Arduino_UNO_R3 -> libs:Arduino_UNO_R3_OVAL
Connections:
- A1 pad 18: Net-(A1-D3) -> Net-(A1-D2)
- SW1 pad 2: Net-(A1-D3) -> Net-(A1-D2)
Routing:
- net Net-(A1-D2): track 54.7 -> 112.5 mm
- net Net-(A1-D3): track 55.7 -> 0.00 mm
