File: sch_pcb/LED Pong.kicad_sch (KiCad schematic)
At the start: 14 parts, among them SW1 SW_Push, SW2 SW_Push

Commit message: update pcb
Parts:
- A1: footprint Module:Arduino_UNO_R3 -> libs:Arduino_UNO_R3_OVAL
Changed lines of the file:
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@@
       (effects (font (size 1.27 1.27)) (justify left))
     )
-    (property "Footprint" "Module:Arduino_UNO_R3" (at 144.78 96.52 0)
+    (property "Footprint" "libs:Arduino_UNO_R3_OVAL" (at 144.78 96.52 0)
       (effects (font (size 1.27 1.27) italic) hide)
     )
